Commit message: change occurences of lh, la, rh, ra, to h1, a1, h0, a1

File: dx_right_dexee_moveit_config/config/gazebo_e3_r3_hand.urdf (robot description, URDF)
Before this commit: robot e3_r3_hand, 21 links, 20 joints
Links:
- removed link rh_F0_J0_link
- removed link rh_F0_base
- removed link rh_F0_distal
- removed link rh_F0_middle
- removed link rh_F0_proximal
- removed link rh_F0_tip
- removed link rh_F1_J0_link
- removed link rh_F1_base
- removed link rh_F1_distal
- removed link rh_F1_middle
- removed link rh_F1_proximal
- removed link rh_F1_tip
- removed link rh_F2_J0_link
- removed link rh_F2_base
- removed link rh_F2_distal
- removed link rh_F2_middle
- removed link rh_F2_proximal
- removed link rh_F2_tip
- removed link rh_end_effector
- removed link rh_hand_base
- added link h0_F0_J0_link, mass 0.13077995; collision mesh filename=package://dx_robot/description/meshes/dx_e3r3_finger/collis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; visual mesh filename=package://dx_robot/description/meshes/dx_e3r3_finger/F0_J0_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
- added link h0_F0_base, mass 0.89937782; collision mesh filename=package://dx_robot/description/meshes/dx_e3r3_finger/collis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; visual mesh filename=package://dx_robot/description/meshes/dx_e3r3_finger/F0_bas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
- added link h0_F0_distal, mass 0.02766365; collision mesh filename=package://dx_robot/description/meshes/dx_e3r3_finger/collis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; visual mesh filename=package://dx_robot/description/meshes/dx_e3r3_finger/F0_dis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
- added link h0_F0_middle, mass 0.05585897; collision mesh filename=package://dx_robot/description/meshes/dx_e3r3_finger/collis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; visual mesh filename=package://dx_robot/description/meshes/dx_e3r3_finger/F0_mid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
- added link h0_F0_proximal, mass 0.09614332; collision mesh filename=package://dx_robot/description/meshes/dx_e3r3_finger/collis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; visual mesh filename=package://dx_robot/description/meshes/dx_e3r3_finger/F0_pro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
- added link h0_F0_tip
- added link h0_F1_J0_link, mass 0.13077995; collision mesh filename=package://dx_robot/description/meshes/dx_e3r3_finger/collis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; visual mesh filename=package://dx_robot/description/meshes/dx_e3r3_finger/F0_J0_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
- added link h0_F1_base, mass 0.89937782; collision mesh filename=package://dx_robot/description/meshes/dx_e3r3_finger/collis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; visual mesh filename=package://dx_robot/description/meshes/dx_e3r3_finger/F0_bas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
- added link h0_F1_distal, mass 0.02766365; collision mesh filename=package://dx_robot/description/meshes/dx_e3r3_finger/collis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; visual mesh filename=package://dx_robot/description/meshes/dx_e3r3_finger/F0_dis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
- added link h0_F1_middle, mass 0.05585897; collision mesh filename=package://dx_robot/description/meshes/dx_e3r3_finger/collis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; visual mesh filename=package://dx_robot/description/meshes/dx_e3r3_finger/F0_mid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
- added link h0_F1_proximal, mass 0.09614332; collision mesh filename=package://dx_robot/description/meshes/dx_e3r3_finger/collis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; visual mesh filename=package://dx_robot/description/meshes/dx_e3r3_finger/F0_pro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
- added link h0_F1_tip
- added link h0_F2_J0_link, mass 0.13077995; collision mesh filename=package://dx_robot/description/meshes/dx_e3r3_finger/collis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; visual mesh filename=package://dx_robot/description/meshes/dx_e3r3_finger/F0_J0_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
- added link h0_F2_base, mass 0.89937782; collision mesh filename=package://dx_robot/description/meshes/dx_e3r3_finger/collis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; visual mesh filename=package://dx_robot/description/meshes/dx_e3r3_finger/F0_bas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
- added link h0_F2_distal, mass 0.02766365; collision mesh filename=package://dx_robot/description/meshes/dx_e3r3_finger/collis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; visual mesh filename=package://dx_robot/description/meshes/dx_e3r3_finger/F0_dis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
- added link h0_F2_middle, mass 0.05585897; collision mesh filename=package://dx_robot/description/meshes/dx_e3r3_finger/collis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; visual mesh filename=package://dx_robot/description/meshes/dx_e3r3_finger/F0_mid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
- added link h0_F2_proximal, mass 0.09614332; collision mesh filename=package://dx_robot/description/meshes/dx_e3r3_finger/collis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; visual mesh filename=package://dx_robot/description/meshes/dx_e3r3_finger/F0_pro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
- added link h0_F2_tip
- added link h0_end_effector
- added link h0_hand_base, mass 0.53506724; collision mesh filename=package://dx_robot/description/meshes/dx_e3r3_finger/collis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; visual mesh filename=package://dx_robot/description/meshes/dx_e3r3_finger/H_Base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
Joints:
- removed joint rh_F0_J0
- removed joint rh_F0_J1
- removed joint rh_F0_J2
- removed joint rh_F0_J3
- removed joint rh_F0_distal_tip
- removed joint rh_F1_J0
- removed joint rh_F1_J1
- removed joint rh_F1_J2
- removed joint rh_F1_J3
- removed joint rh_F1_distal_tip
- removed joint rh_F2_J0
- removed joint rh_F2_J1
- removed joint rh_F2_J2
- removed joint rh_F2_J3
- removed joint rh_F2_distal_tip
- removed joint rh_ee_fixed_joint
- removed joint rh_world_joint
- removed joint rh_world_joint_F0
- removed joint rh_world_joint_F1
- removed joint rh_world_joint_F2
- added joint h0_F0_J0: type revolute, parent h0_F0_base, child h0_F0_J0_link, origin xyz=0 -0.14073 -0.051327 rpy=2.0944 0 0, axis 0 -1 0, limit lower=-0.8727 upper=0.8727 effort=1.5 velocity=3.1415
- added joint h0_F0_J1: type revolute, parent h0_F0_J0_link, child h0_F0_proximal, origin xyz=0 0.0765883365730207 0.0299999999999999 rpy=0 0 0, axis 1 0 0, limit lower=-1.396 upper=0.785 effort=1.2 velocity=3.1415
- added joint h0_F0_J2: type revolute, parent h0_F0_proximal, child h0_F0_middle, origin xyz=0 0 0.05 rpy=0 0 0, axis 1 0 0, limit lower=0 upper=1.396 effort=0.7 velocity=3.1415
- added joint h0_F0_J3: type revolute, parent h0_F0_middle, child h0_F0_distal, origin xyz=0 0 0.035 rpy=0 0 0, axis 1 0 0, limit lower=-0.523 upper=1.485 effort=0.35 velocity=3.1415
- added joint h0_F0_distal_tip: type fixed, parent h0_F0_distal, child h0_F0_tip, origin xyz=0 0.003 0.033 rpy=0 0 0
- added joint h0_F1_J0: type revolute, parent h0_F1_base, child h0_F1_J0_link, origin xyz=0 -0.14073 -0.051327 rpy=2.0944 0 0, axis 0 -1 0, limit lower=-0.8727 upper=0.8727 effort=1.5 velocity=3.1415
- added joint h0_F1_J1: type revolute, parent h0_F1_J0_link, child h0_F1_proximal, origin xyz=0 0.0765883365730207 0.0299999999999999 rpy=0 0 0, axis 1 0 0, limit lower=-1.396 upper=0.785 effort=1.2 velocity=3.1415
- added joint h0_F1_J2: type revolute, parent h0_F1_proximal, child h0_F1_middle, origin xyz=0 0 0.05 rpy=0 0 0, axis 1 0 0, limit lower=0 upper=1.396 effort=0.7 velocity=3.1415
- added joint h0_F1_J3: type revolute, parent h0_F1_middle, child h0_F1_distal, origin xyz=0 0 0.035 rpy=0 0 0, axis 1 0 0, limit lower=-0.523 upper=1.485 effort=0.35 velocity=3.1415
- added joint h0_F1_distal_tip: type fixed, parent h0_F1_distal, child h0_F1_tip, origin xyz=0 0.003 0.033 rpy=0 0 0
- added joint h0_F2_J0: type revolute, parent h0_F2_base, child h0_F2_J0_link, origin xyz=0 -0.14073 -0.051327 rpy=2.0944 0 0, axis 0 -1 0, limit lower=-0.8727 upper=0.8727 effort=1.5 velocity=3.1415
- added joint h0_F2_J1: type revolute, parent h0_F2_J0_link, child h0_F2_proximal, origin xyz=0 0.0765883365730207 0.0299999999999999 rpy=0 0 0, axis 1 0 0, limit lower=-1.396 upper=0.785 effort=1.2 velocity=3.1415
- added joint h0_F2_J2: type revolute, parent h0_F2_proximal, child h0_F2_middle, origin xyz=0 0 0.05 rpy=0 0 0, axis 1 0 0, limit lower=0 upper=1.396 effort=0.7 velocity=3.1415
- added joint h0_F2_J3: type revolute, parent h0_F2_middle, child h0_F2_distal, origin xyz=0 0 0.035 rpy=0 0 0, axis 1 0 0, limit lower=-0.523 upper=1.485 effort=0.35 velocity=3.1415
- added joint h0_F2_distal_tip: type fixed, parent h0_F2_distal, child h0_F2_tip, origin xyz=0 0.003 0.033 rpy=0 0 0
- added joint h0_ee_fixed_joint: type fixed, parent h0_hand_base, child h0_end_effector, origin xyz=0.0 0.0 0.25 rpy=0.0 0.0 0.0
- added joint h0_world_joint: type fixed, parent world, child h0_hand_base
- added joint h0_world_joint_F0: type fixed, parent h0_hand_base, child h0_F0_base, origin xyz=0 0.05 0.017 rpy=-1.5707 0 0
- added joint h0_world_joint_F1: type fixed, parent h0_hand_base, child h0_F1_base, origin xyz=0.0384 -0.0287 0.017 rpy=-1.5707 0 -2.8159
- added joint h0_world_joint_F2: type fixed, parent h0_hand_base, child h0_F2_base, origin xyz=-0.0384 -0.02870 0.017 rpy=-1.5707 0 2.8159

File: dx_right_dexee_ur_moveit_config/config/gazebo_ur_dex.urdf (robot description, URDF)
Before this commit: robot ur_dex, 31 links, 30 joints
Links:
- removed link ra_base
- removed link ra_base_link
- removed link ra_base_link_inertia
- removed link ra_flange
- removed link ra_forearm_link
- removed link ra_shoulder_link
- removed link ra_tool0
- removed link ra_upper_arm_link
- removed link ra_wrist_1_link
- removed link ra_wrist_2_link
- removed link ra_wrist_3_link
- removed link rh_F0_J0_link
- removed link rh_F0_base
- removed link rh_F0_distal
- removed link rh_F0_middle
- removed link rh_F0_proximal
- removed link rh_F0_tip
- removed link rh_F1_J0_link
- removed link rh_F1_base
- removed link rh_F1_distal
- removed link rh_F1_middle
- removed link rh_F1_proximal
- removed link rh_F1_tip
- removed link rh_F2_J0_link
- removed link rh_F2_base
- removed link rh_F2_distal
- removed link rh_F2_middle
- removed link rh_F2_proximal
- removed link rh_F2_tip
- removed link rh_hand_base
- added link a0_base
- added link a0_base_link
- added link a0_base_link_inertia, mass 4.0; collision mesh filename=package://ur_description/meshes/ur10e/collision/base.stl; visual mesh filename=package://ur_description/meshes/ur10e/visual/base.dae
- added link a0_flange
- added link a0_forearm_link, mass 3.87; collision mesh filename=package://ur_description/meshes/ur10e/collision/forearm.stl; visual mesh filename=package://ur_description/meshes/ur10e/visual/forearm.dae
- added link a0_shoulder_link, mass 7.778; collision mesh filename=package://ur_description/meshes/ur10e/collision/shoulder.stl; visual mesh filename=package://ur_description/meshes/ur10e/visual/shoulder.dae
- added link a0_tool0
- added link a0_upper_arm_link, mass 12.93; collision mesh filename=package://ur_description/meshes/ur10e/collision/upperarm.stl; visual mesh filename=package://ur_description/meshes/ur10e/visual/upperarm.dae
- added link a0_wrist_1_link, mass 1.96; collision mesh filename=package://ur_description/meshes/ur10e/collision/wrist1.stl; visual mesh filename=package://ur_description/meshes/ur10e/visual/wrist1.dae
- added link a0_wrist_2_link, mass 1.96; collision mesh filename=package://ur_description/meshes/ur10e/collision/wrist2.stl; visual mesh filename=package://ur_description/meshes/ur10e/visual/wrist2.dae
- added link a0_wrist_3_link, mass 0.202; collision mesh filename=package://ur_description/meshes/ur10e/collision/wrist3.stl; visual mesh filename=package://ur_description/meshes/ur10e/visual/wrist3.dae
- added link h0_F0_J0_link, mass 0.13077995; collision mesh filename=package://dx_robot/description/meshes/dx_e3r3_finger/collis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; visual mesh filename=package://dx_robot/description/meshes/dx_e3r3_finger/F0_J0_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
- added link h0_F0_base, mass 0.89937782; collision mesh filename=package://dx_robot/description/meshes/dx_e3r3_finger/collis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; visual mesh filename=package://dx_robot/description/meshes/dx_e3r3_finger/F0_bas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
- added link h0_F0_distal, mass 0.02766365; collision mesh filename=package://dx_robot/description/meshes/dx_e3r3_finger/collis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; visual mesh filename=package://dx_robot/description/meshes/dx_e3r3_finger/F0_dis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
- added link h0_F0_middle, mass 0.05585897; collision mesh filename=package://dx_robot/description/meshes/dx_e3r3_finger/collis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; visual mesh filename=package://dx_robot/description/meshes/dx_e3r3_finger/F0_mid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
- added link h0_F0_proximal, mass 0.09614332; collision mesh filename=package://dx_robot/description/meshes/dx_e3r3_finger/collis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; visual mesh filename=package://dx_robot/description/meshes/dx_e3r3_finger/F0_pro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
- added link h0_F0_tip
- added link h0_F1_J0_link, mass 0.13077995; collision mesh filename=package://dx_robot/description/meshes/dx_e3r3_finger/collis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; visual mesh filename=package://dx_robot/description/meshes/dx_e3r3_finger/F0_J0_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
- added link h0_F1_base, mass 0.89937782; collision mesh filename=package://dx_robot/description/meshes/dx_e3r3_finger/collis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; visual mesh filename=package://dx_robot/description/meshes/dx_e3r3_finger/F0_bas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
- added link h0_F1_distal, mass 0.02766365; collision mesh filename=package://dx_robot/description/meshes/dx_e3r3_finger/collis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; visual mesh filename=package://dx_robot/description/meshes/dx_e3r3_finger/F0_dis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
- added link h0_F1_middle, mass 0.05585897; collision mesh filename=package://dx_robot/description/meshes/dx_e3r3_finger/collis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; visual mesh filename=package://dx_robot/description/meshes/dx_e3r3_finger/F0_mid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
- added link h0_F1_proximal, mass 0.09614332; collision mesh filename=package://dx_robot/description/meshes/dx_e3r3_finger/collis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; visual mesh filename=package://dx_robot/description/meshes/dx_e3r3_finger/F0_pro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
- added link h0_F1_tip
- added link h0_F2_J0_link, mass 0.13077995; collision mesh filename=package://dx_robot/description/meshes/dx_e3r3_finger/collis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; visual mesh filename=package://dx_robot/description/meshes/dx_e3r3_finger/F0_J0_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
- added link h0_F2_base, mass 0.89937782; collision mesh filename=package://dx_robot/description/meshes/dx_e3r3_finger/collis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; visual mesh filename=package://dx_robot/description/meshes/dx_e3r3_finger/F0_bas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
- added link h0_F2_distal, mass 0.02766365; collision mesh filename=package://dx_robot/description/meshes/dx_e3r3_finger/collis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; visual mesh filename=package://dx_robot/description/meshes/dx_e3r3_finger/F0_dis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
- added link h0_F2_middle, mass 0.05585897; collision mesh filename=package://dx_robot/description/meshes/dx_e3r3_finger/collis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; visual mesh filename=package://dx_robot/description/meshes/dx_e3r3_finger/F0_mid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
- added link h0_F2_proximal, mass 0.09614332; collision mesh filename=package://dx_robot/description/meshes/dx_e3r3_finger/collis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; visual mesh filename=package://dx_robot/description/meshes/dx_e3r3_finger/F0_pro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
- added link h0_F2_tip
- added link h0_hand_base, mass 0.53506724; collision mesh filename=package://dx_robot/description/meshes/dx_e3r3_finger/collis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; visual mesh filename=package://dx_robot/description/meshes/dx_e3r3_finger/H_Base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
Joints:
- removed joint ra_arm_to_hand
- removed joint ra_base_link-base_fixed_joint
- removed joint ra_base_link-base_link_inertia
- removed joint ra_elbow_joint
- removed joint ra_flange-tool0
- removed joint ra_shoulder_lift_joint
- removed joint ra_shoulder_pan_joint
- removed joint ra_wrist_1_joint
- removed joint ra_wrist_2_joint
- removed joint ra_wrist_3-flange
- removed joint ra_wrist_3_joint
- removed joint rh_F0_J0
- removed joint rh_F0_J1
- removed joint rh_F0_J2
- removed joint rh_F0_J3
- removed joint rh_F0_distal_tip
- removed joint rh_F1_J0
- removed joint rh_F1_J1
- removed joint rh_F1_J2
- removed joint rh_F1_J3
- removed joint rh_F1_distal_tip
- removed joint rh_F2_J0
- removed joint rh_F2_J1
- removed joint rh_F2_J2
- removed joint rh_F2_J3
- removed joint rh_F2_distal_tip
- removed joint rh_world_joint_F0
- removed joint rh_world_joint_F1
- removed joint rh_world_joint_F2
- added joint a0_arm_to_hand: type fixed, parent a0_flange, child h0_hand_base, origin xyz=0.0 0.0 0.0 rpy=1.5707963267948966 3.141592653589793 1.5707963267948966
- added joint a0_base_link-base_fixed_joint: type fixed, parent a0_base_link, child a0_base, origin xyz=0 0 0 rpy=0 0 3.141592653589793
- added joint a0_base_link-base_link_inertia: type fixed, parent a0_base_link, child a0_base_link_inertia, origin xyz=0 0 0 rpy=0 0 3.141592653589793
- added joint a0_elbow_joint: type revolute, parent a0_upper_arm_link, child a0_forearm_link, origin xyz=-0.6127 0 0 rpy=0 0 0, axis 0 0 1, limit lower=-3.141592653589793 upper=3.141592653589793 effort=150.0 velocity=3.141592653589793
- added joint a0_flange-tool0: type fixed, parent a0_flange, child a0_tool0, origin xyz=0 0 0 rpy=1.5707963267948966 0 1.5707963267948966
- added joint a0_shoulder_lift_joint: type revolute, parent a0_shoulder_link, child a0_upper_arm_link, origin xyz=0 0 0 rpy=1.570796327 0 0, axis 0 0 1, limit lower=-6.283185307179586 upper=6.283185307179586 effort=330.0 velocity=2.0943951023931953
- added joint a0_shoulder_pan_joint: type revolute, parent a0_base_link_inertia, child a0_shoulder_link, origin xyz=0 0 0.1807 rpy=0 0 0, axis 0 0 1, limit lower=-6.283185307179586 upper=6.283185307179586 effort=330.0 velocity=2.0943951023931953
- added joint a0_wrist_1_joint: type revolute, parent a0_forearm_link, child a0_wrist_1_link, origin xyz=-0.57155 0 0.17415 rpy=0 0 0, axis 0 0 1, limit lower=-6.283185307179586 upper=6.283185307179586 effort=56.0 velocity=3.141592653589793
- added joint a0_wrist_2_joint: type revolute, parent a0_wrist_1_link, child a0_wrist_2_link, origin xyz=0 -0.11985 -2.458164590756244e-11 rpy=1.570796327 0 0, axis 0 0 1, limit lower=-6.283185307179586 upper=6.283185307179586 effort=56.0 velocity=3.141592653589793
- added joint a0_wrist_3-flange: type fixed, parent a0_wrist_3_link, child a0_flange, origin xyz=0 0 0 rpy=0 -1.5707963267948966 -1.5707963267948966
- added joint a0_wrist_3_joint: type revolute, parent a0_wrist_2_link, child a0_wrist_3_link, origin xyz=0 0.11655 -2.390480459346185e-11 rpy=1.570796326589793 3.141592653589793 3.141592653589793, axis 0 0 1, limit lower=-6.283185307179586 upper=6.283185307179586 effort=56.0 velocity=3.141592653589793
- added joint h0_F0_J0: type revolute, parent h0_F0_base, child h0_F0_J0_link, origin xyz=0 -0.14073 -0.051327 rpy=2.0944 0 0, axis 0 -1 0, limit lower=-0.8727 upper=0.8727 effort=1.5 velocity=2
- added joint h0_F0_J1: type revolute, parent h0_F0_J0_link, child h0_F0_proximal, origin xyz=0 0.0765883365730207 0.0299999999999999 rpy=0 0 0, axis 1 0 0, limit lower=-1.396 upper=0.785 effort=1.2 velocity=2
- added joint h0_F0_J2: type revolute, parent h0_F0_proximal, child h0_F0_middle, origin xyz=0 0 0.05 rpy=0 0 0, axis 1 0 0, limit lower=0 upper=1.396 effort=0.7 velocity=2
- added joint h0_F0_J3: type revolute, parent h0_F0_middle, child h0_F0_distal, origin xyz=0 0 0.035 rpy=0 0 0, axis 1 0 0, limit lower=-0.523 upper=1.485 effort=0.35 velocity=0.2
- added joint h0_F0_distal_tip: type fixed, parent h0_F0_distal, child h0_F0_tip, origin xyz=0 0.003 0.033 rpy=0 0 0
- added joint h0_F1_J0: type revolute, parent h0_F1_base, child h0_F1_J0_link, origin xyz=0 -0.14073 -0.051327 rpy=2.0944 0 0, axis 0 -1 0, limit lower=-0.8727 upper=0.8727 effort=1.5 velocity=2
- added joint h0_F1_J1: type revolute, parent h0_F1_J0_link, child h0_F1_proximal, origin xyz=0 0.0765883365730207 0.0299999999999999 rpy=0 0 0, axis 1 0 0, limit lower=-1.396 upper=0.785 effort=1.2 velocity=2
- added joint h0_F1_J2: type revolute, parent h0_F1_proximal, child h0_F1_middle, origin xyz=0 0 0.05 rpy=0 0 0, axis 1 0 0, limit lower=0 upper=1.396 effort=0.7 velocity=2
- added joint h0_F1_J3: type revolute, parent h0_F1_middle, child h0_F1_distal, origin xyz=0 0 0.035 rpy=0 0 0, axis 1 0 0, limit lower=-0.523 upper=1.485 effort=0.35 velocity=0.2
- added joint h0_F1_distal_tip: type fixed, parent h0_F1_distal, child h0_F1_tip, origin xyz=0 0.003 0.033 rpy=0 0 0
- added joint h0_F2_J0: type revolute, parent h0_F2_base, child h0_F2_J0_link, origin xyz=0 -0.14073 -0.051327 rpy=2.0944 0 0, axis 0 -1 0, limit lower=-0.8727 upper=0.8727 effort=1.5 velocity=2
- added joint h0_F2_J1: type revolute, parent h0_F2_J0_link, child h0_F2_proximal, origin xyz=0 0.0765883365730207 0.0299999999999999 rpy=0 0 0, axis 1 0 0, limit lower=-1.396 upper=0.785 effort=1.2 velocity=2
- added joint h0_F2_J2: type revolute, parent h0_F2_proximal, child h0_F2_middle, origin xyz=0 0 0.05 rpy=0 0 0, axis 1 0 0, limit lower=0 upper=1.396 effort=0.7 velocity=2
- added joint h0_F2_J3: type revolute, parent h0_F2_middle, child h0_F2_distal, origin xyz=0 0 0.035 rpy=0 0 0, axis 1 0 0, limit lower=-0.523 upper=1.485 effort=0.35 velocity=0.2
- added joint h0_F2_distal_tip: type fixed, parent h0_F2_distal, child h0_F2_tip, origin xyz=0 0.003 0.033 rpy=0 0 0
- added joint h0_world_joint_F0: type fixed, parent h0_hand_base, child h0_F0_base, origin xyz=0 0.05 0.017 rpy=-1.5707 0 0
- added joint h0_world_joint_F1: type fixed, parent h0_hand_base, child h0_F1_base, origin xyz=0.0384 -0.0287 0.017 rpy=-1.5707 0 -2.8159
- added joint h0_world_joint_F2: type fixed, parent h0_hand_base, child h0_F2_base, origin xyz=-0.0384 -0.02870 0.017 rpy=-1.5707 0 2.8159
- joint world_joint: child ra_base_link -> a0_base_link
