Commit message: addressing pr comments

File: dx_launch/description/bimanual_dexee_ur.urdf.xacro (robot description, xacro)
@@ -100,5 +100,5 @@
       <parent link="world"/>
       <child link="a1_base_link"/>
-      <origin xyz="0.0 $(arg initial_y_1) $(arg initial_z_1)" rpy="0.0 0.0 ${$(arg initial_yaw_1) + pi}"/>
+      <origin xyz="0.0 $(arg initial_y_1) $(arg initial_z_1)" rpy="0.0 0.0 $(arg initial_yaw_1)"/>
   </joint>
   <xacro:if value="$(arg mounting_plate)">

Commit message: Fix dexee rotation on arm

File: dx_launch/description/bimanual_dexee_ur.urdf.xacro (robot description, xacro)
@@ -73,5 +73,5 @@
     <xacro:include filename="$(find dx_description)/xacros/mounting_plates/$(arg mounting_plate_name).xacro" />
     <xacro:macro_e3r3_mounting_plate prefix="h0_" parent="a0_flange" mounted_tool="h0_hand_base" >
-      <origin xyz="0.0 0.0 0.0" rpy="${pi/2.0} ${3.0*pi/4.0} ${pi/2.0}"/>
+      <origin xyz="0.0 0.0 0.0" rpy="${pi/2.0} ${0} ${pi/2.0}"/>
     </xacro:macro_e3r3_mounting_plate>
   </xacro:if>
@@ -80,5 +80,5 @@
       <parent link="a0_flange"/>
       <child link="h0_hand_base"/>
-      <origin xyz="0.0 0.0 0.0" rpy="${pi/2.0} ${3.0*pi/4.0} ${pi/2.0}"/>
+      <origin xyz="0.0 0.0 0.0" rpy="${pi/2.0} ${0} ${pi/2.0}"/>
     </joint>
   </xacro:unless>
@@ -104,5 +104,5 @@
   <xacro:if value="$(arg mounting_plate)">
     <xacro:macro_e3r3_mounting_plate prefix="h1_" parent="a1_flange" mounted_tool="h1_hand_base" >
-      <origin xyz="0.0 0.0 0.0" rpy="${pi/2.0} ${-3.0*pi/4.0} ${pi/2.0}"/>
+      <origin xyz="0.0 0.0 0.0" rpy="${pi/2.0} ${0} ${pi/2.0}"/>
     </xacro:macro_e3r3_mounting_plate>
   </xacro:if>
@@ -111,5 +111,5 @@
       <parent link="a1_flange"/>
       <child link="h1_hand_base"/>
-      <origin xyz="0.0 0.0 0.0" rpy="${pi/2.0} ${-3.0*pi/4.0} ${pi/2.0}"/>
+      <origin xyz="0.0 0.0 0.0" rpy="${pi/2.0} ${0} ${pi/2.0}"/>
     </joint>
   </xacro:unless>

Commit message: 45 deg mounting plate

File: dx_launch/description/bimanual_dexee_ur.urdf.xacro (robot description, xacro)
@@ -73,5 +73,5 @@
     <xacro:include filename="$(find dx_description)/xacros/mounting_plates/$(arg mounting_plate_name).xacro" />
     <xacro:macro_e3r3_mounting_plate prefix="h0_" parent="a0_flange" mounted_tool="h0_hand_base" >
-      <origin xyz="0.0 0.0 0.0" rpy="${pi/2.0} ${0} ${pi/2.0}"/>
+      <origin xyz="0.0 0.0 0.0" rpy="${pi/2.0} ${3.0*pi/4.0} ${pi/2.0}"/>
     </xacro:macro_e3r3_mounting_plate>
   </xacro:if>
@@ -80,5 +80,5 @@
       <parent link="a0_flange"/>
       <child link="h0_hand_base"/>
-      <origin xyz="0.0 0.0 0.0" rpy="${pi/2.0} ${0} ${pi/2.0}"/>
+      <origin xyz="0.0 0.0 0.0" rpy="${pi/2.0} ${3.0*pi/4.0} ${pi/2.0}"/>
     </joint>
   </xacro:unless>
@@ -104,5 +104,5 @@
   <xacro:if value="$(arg mounting_plate)">
     <xacro:macro_e3r3_mounting_plate prefix="h1_" parent="a1_flange" mounted_tool="h1_hand_base" >
-      <origin xyz="0.0 0.0 0.0" rpy="${pi/2.0} ${0} ${pi/2.0}"/>
+      <origin xyz="0.0 0.0 0.0" rpy="${pi/2.0} ${3.0*pi/4.0} ${pi/2.0}"/>
     </xacro:macro_e3r3_mounting_plate>
   </xacro:if>
@@ -111,5 +111,5 @@
       <parent link="a1_flange"/>
       <child link="h1_hand_base"/>
-      <origin xyz="0.0 0.0 0.0" rpy="${pi/2.0} ${0} ${pi/2.0}"/>
+      <origin xyz="0.0 0.0 0.0" rpy="${pi/2.0} ${3.0*pi/4.0} ${pi/2.0}"/>
     </joint>
   </xacro:unless>

Commit message: invert other hand

File: dx_launch/description/bimanual_dexee_ur.urdf.xacro (robot description, xacro)
@@ -104,5 +104,5 @@
   <xacro:if value="$(arg mounting_plate)">
     <xacro:macro_e3r3_mounting_plate prefix="h1_" parent="a1_flange" mounted_tool="h1_hand_base" >
-      <origin xyz="0.0 0.0 0.0" rpy="${pi/2.0} ${3.0*pi/4.0} ${pi/2.0}"/>
+      <origin xyz="0.0 0.0 0.0" rpy="${pi/2.0} ${-3.0*pi/4.0} ${pi/2.0}"/>
     </xacro:macro_e3r3_mounting_plate>
   </xacro:if>
@@ -111,5 +111,5 @@
       <parent link="a1_flange"/>
       <child link="h1_hand_base"/>
-      <origin xyz="0.0 0.0 0.0" rpy="${pi/2.0} ${3.0*pi/4.0} ${pi/2.0}"/>
+      <origin xyz="0.0 0.0 0.0" rpy="${pi/2.0} ${-3.0*pi/4.0} ${pi/2.0}"/>
     </joint>
   </xacro:unless>

Commit message: fix mounting plate orientation for left arm

File: dx_launch/description/bimanual_dexee_ur.urdf.xacro (robot description, xacro)
@@ -104,5 +104,5 @@
   <xacro:if value="$(arg mounting_plate)">
     <xacro:macro_e3r3_mounting_plate prefix="h1_" parent="a1_flange" mounted_tool="h1_hand_base" >
-      <origin xyz="0.0 0.0 0.0" rpy="${pi/2.0} ${-3.0*pi/4.0} ${pi/2.0}"/>
+      <origin xyz="0.0 0.0 0.0" rpy="${pi/2.0} ${3.0*pi/4.0} ${pi/2.0}"/>
     </xacro:macro_e3r3_mounting_plate>
   </xacro:if>
@@ -111,5 +111,5 @@
       <parent link="a1_flange"/>
       <child link="h1_hand_base"/>
-      <origin xyz="0.0 0.0 0.0" rpy="${pi/2.0} ${-3.0*pi/4.0} ${pi/2.0}"/>
+      <origin xyz="0.0 0.0 0.0" rpy="${pi/2.0} ${3.0*pi/4.0} ${pi/2.0}"/>
     </joint>
   </xacro:unless>
