Commit message: Fix paths

File: dx_dexee_0_moveit_config/config/gazebo_e3_r3_hand.urdf (robot description, URDF)
Before this commit: robot e3_r3_hand, 21 links, 20 joints
Links:
- link h0_F0_J0_link: geometry collision mesh filename=package://dx_description/meshes/dx_e3r3_finger/collision/F0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; visual mesh filename=package://dx_description/meshes/dx_e3r3_finger/F0_J0_link.S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
- link h0_F0_base: geometry collision mesh filename=package://dx_description/meshes/dx_e3r3_finger/collision/F0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; visual mesh filename=package://dx_description/meshes/dx_e3r3_finger/F0_base.STL
- link h0_F0_distal: geometry collision mesh filename=package://dx_description/meshes/dx_e3r3_finger/collision/F0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; visual mesh filename=package://dx_description/meshes/dx_e3r3_finger/F0_distal.STL
- link h0_F0_middle: geometry collision mesh filename=package://dx_description/meshes/dx_e3r3_finger/collision/F0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; visual mesh filename=package://dx_description/meshes/dx_e3r3_finger/F0_middle.STL
- link h0_F0_proximal: geometry collision mesh filename=package://dx_description/meshes/dx_e3r3_finger/collision/F0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; visual mesh filename=package://dx_description/meshes/dx_e3r3_finger/F0_proximal.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
- link h0_F1_J0_link: geometry collision mesh filename=package://dx_description/meshes/dx_e3r3_finger/collision/F0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; visual mesh filename=package://dx_description/meshes/dx_e3r3_finger/F0_J0_link.S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
- link h0_F1_base: geometry collision mesh filename=package://dx_description/meshes/dx_e3r3_finger/collision/F0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; visual mesh filename=package://dx_description/meshes/dx_e3r3_finger/F0_base.STL
- link h0_F1_distal: geometry collision mesh filename=package://dx_description/meshes/dx_e3r3_finger/collision/F0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; visual mesh filename=package://dx_description/meshes/dx_e3r3_finger/F0_distal.STL
- link h0_F1_middle: geometry collision mesh filename=package://dx_description/meshes/dx_e3r3_finger/collision/F0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; visual mesh filename=package://dx_description/meshes/dx_e3r3_finger/F0_middle.STL
- link h0_F1_proximal: geometry collision mesh filename=package://dx_description/meshes/dx_e3r3_finger/collision/F0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; visual mesh filename=package://dx_description/meshes/dx_e3r3_finger/F0_proximal.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
- link h0_F2_J0_link: geometry collision mesh filename=package://dx_description/meshes/dx_e3r3_finger/collision/F0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; visual mesh filename=package://dx_description/meshes/dx_e3r3_finger/F0_J0_link.S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
- link h0_F2_base: geometry collision mesh filename=package://dx_description/meshes/dx_e3r3_finger/collision/F0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; visual mesh filename=package://dx_description/meshes/dx_e3r3_finger/F0_base.STL
- link h0_F2_distal: geometry collision mesh filename=package://dx_description/meshes/dx_e3r3_finger/collision/F0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; visual mesh filename=package://dx_description/meshes/dx_e3r3_finger/F0_distal.STL
- link h0_F2_middle: geometry collision mesh filename=package://dx_description/meshes/dx_e3r3_finger/collision/F0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; visual mesh filename=package://dx_description/meshes/dx_e3r3_finger/F0_middle.STL
- link h0_F2_proximal: geometry collision mesh filename=package://dx_description/meshes/dx_e3r3_finger/collision/F0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; visual mesh filename=package://dx_description/meshes/dx_e3r3_finger/F0_proximal.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
- link h0_hand_base: geometry collision mesh filename=package://dx_description/meshes/dx_e3r3_finger/collision/Ha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; visual mesh filename=package://dx_description/meshes/dx_e3r3_finger/H_Base.STL

File: dx_dexee_0_ur_moveit_config/config/gazebo_ur_dex.urdf (robot description, URDF)
Before this commit: robot ur_dex, 31 links, 30 joints
Links:
- link h0_F0_J0_link: geometry collision mesh filename=package://dx_description/meshes/dx_e3r3_finger/collision/F0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; visual mesh filename=package://dx_description/meshes/dx_e3r3_finger/F0_J0_link.S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
- link h0_F0_base: geometry collision mesh filename=package://dx_description/meshes/dx_e3r3_finger/collision/F0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; visual mesh filename=package://dx_description/meshes/dx_e3r3_finger/F0_base.STL
- link h0_F0_distal: geometry collision mesh filename=package://dx_description/meshes/dx_e3r3_finger/collision/F0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; visual mesh filename=package://dx_description/meshes/dx_e3r3_finger/F0_distal.STL
- link h0_F0_middle: geometry collision mesh filename=package://dx_description/meshes/dx_e3r3_finger/collision/F0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; visual mesh filename=package://dx_description/meshes/dx_e3r3_finger/F0_middle.STL
- link h0_F0_proximal: geometry collision mesh filename=package://dx_description/meshes/dx_e3r3_finger/collision/F0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; visual mesh filename=package://dx_description/meshes/dx_e3r3_finger/F0_proximal.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
- link h0_F1_J0_link: geometry collision mesh filename=package://dx_description/meshes/dx_e3r3_finger/collision/F0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; visual mesh filename=package://dx_description/meshes/dx_e3r3_finger/F0_J0_link.S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
- link h0_F1_base: geometry collision mesh filename=package://dx_description/meshes/dx_e3r3_finger/collision/F0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; visual mesh filename=package://dx_description/meshes/dx_e3r3_finger/F0_base.STL
- link h0_F1_distal: geometry collision mesh filename=package://dx_description/meshes/dx_e3r3_finger/collision/F0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; visual mesh filename=package://dx_description/meshes/dx_e3r3_finger/F0_distal.STL
- link h0_F1_middle: geometry collision mesh filename=package://dx_description/meshes/dx_e3r3_finger/collision/F0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; visual mesh filename=package://dx_description/meshes/dx_e3r3_finger/F0_middle.STL
- link h0_F1_proximal: geometry collision mesh filename=package://dx_description/meshes/dx_e3r3_finger/collision/F0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; visual mesh filename=package://dx_description/meshes/dx_e3r3_finger/F0_proximal.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
- link h0_F2_J0_link: geometry collision mesh filename=package://dx_description/meshes/dx_e3r3_finger/collision/F0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; visual mesh filename=package://dx_description/meshes/dx_e3r3_finger/F0_J0_link.S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
- link h0_F2_base: geometry collision mesh filename=package://dx_description/meshes/dx_e3r3_finger/collision/F0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; visual mesh filename=package://dx_description/meshes/dx_e3r3_finger/F0_base.STL
- link h0_F2_distal: geometry collision mesh filename=package://dx_description/meshes/dx_e3r3_finger/collision/F0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; visual mesh filename=package://dx_description/meshes/dx_e3r3_finger/F0_distal.STL
- link h0_F2_middle: geometry collision mesh filename=package://dx_description/meshes/dx_e3r3_finger/collision/F0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; visual mesh filename=package://dx_description/meshes/dx_e3r3_finger/F0_middle.STL
- link h0_F2_proximal: geometry collision mesh filename=package://dx_description/meshes/dx_e3r3_finger/collision/F0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; visual mesh filename=package://dx_description/meshes/dx_e3r3_finger/F0_proximal.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
- link h0_hand_base: geometry collision mesh filename=package://dx_description/meshes/dx_e3r3_finger/collision/Ha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; visual mesh filename=package://dx_description/meshes/dx_e3r3_finger/H_Base.STL

File: dx_launch/description/0x02000105.urdf.xacro (robot description, xacro)
@@ -2,5 +2,5 @@
 <!--
  Software License Agreement (BSD License)
- Copyright © 2024-2025 belongs to Shadow Robot Company Ltd.
+ Copyright © 2024-2026 belongs to Shadow Robot Company Ltd.
  All rights reserved.
  Redistribution and use in source and binary forms, with or without modification,
@@ -25,5 +25,5 @@
 -->
 <robot name="e3_r3_hand" xmlns:xacro="http://www.ros.org/wiki/xacro">
-  <xacro:include filename="$(find dx_robot)/description/robot/0x02000105.xacro" />
+  <xacro:include filename="$(find dx_description)/robot/0x02000105.xacro" />
   <xacro:arg name="prefix" default="" />
   <xacro:arg name="robot_system_id" default="" />

File: dx_launch/description/dexee_ur.urdf.xacro (robot description, xacro)
@@ -2,5 +2,5 @@
 <!--
  Software License Agreement (BSD License)
- Copyright © 2024-2025 belongs to Shadow Robot Company Ltd.
+ Copyright © 2024-2026 belongs to Shadow Robot Company Ltd.
  All rights reserved.
  Redistribution and use in source and binary forms, with or without modification,
@@ -55,5 +55,5 @@
       <xacro:ur5_robot prefix="$(arg arm_prefix)_" transmission_hw_interface="$(arg transmission_hw_interface)" kinematics_parameters_file="$(arg kinematics_config)"/>
   </xacro:if>
-  <xacro:include filename="$(find dx_robot)/description/robot/$(arg hand_type).xacro" />
+  <xacro:include filename="$(find dx_description)/robot/$(arg hand_type).xacro" />
   <xacro:e3_r3_hand prefix="$(arg hand_prefix)_" />
   <joint name="world_joint" type="fixed">
@@ -63,5 +63,5 @@
   </joint>
   <xacro:if value="$(arg mounting_plate)">
-    <xacro:include filename="$(find dx_robot)/description/xacros/mounting_plates/$(arg mounting_plate_name).xacro" />
+    <xacro:include filename="$(find dx_description)/xacros/mounting_plates/$(arg mounting_plate_name).xacro" />
     <xacro:macro_e3r3_mounting_plate prefix="$(arg hand_prefix)_" parent="$(arg arm_prefix)_flange" mounted_tool="$(arg hand_prefix)_hand_base" >
       <origin xyz="0.0 0.0 0.0" rpy="${pi/2.0} ${3.0*pi/4.0} ${pi/2.0}"/>

Commit message: fixed mesh paths and bimanual xacro and launch file

File: dx_dexee_0_moveit_config/config/gazebo_e3_r3_hand.urdf (robot description, URDF)
Before this commit: robot e3_r3_hand, 21 links, 20 joints
Links:
- link h0_hand_base: geometry collision mesh filename=package://dx_description/meshes/hand_bases/collision/Config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; visual mesh filename=package://dx_description/meshes/hand_bases/Config_1_Hand_Ba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

File: dx_dexee_0_ur_moveit_config/config/gazebo_ur_dex.urdf (robot description, URDF)
Before this commit: robot ur_dex, 31 links, 30 joints
Links:
- link h0_hand_base: geometry collision mesh filename=package://dx_description/meshes/hand_bases/collision/Config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; visual mesh filename=package://dx_description/meshes/hand_bases/Config_1_Hand_Ba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

File: dx_dexee_config_2_lh_moveit_config/config/gazebo_dexee_config_2_left_hand.urdf (robot description, URDF)
Before this commit: robot dexee_config_2_left_hand, 21 links, 20 joints
Links:
- link hand_base: geometry collision mesh filename=package://dx_description/meshes/hand_bases/collision/Config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; visual mesh filename=package://dx_description/meshes/hand_bases/Config_2_Left_Ha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

File: dx_dexee_config_2_rh_moveit_config/config/gazebo_dexee_config_2_right_hand.urdf (robot description, URDF)
Before this commit: robot dexee_config_2_right_hand, 21 links, 20 joints
Links:
- link hand_base: geometry collision mesh filename=package://dx_description/meshes/hand_bases/collision/Config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; visual mesh filename=package://dx_description/meshes/hand_bases/Config_2_Right_H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

File: dx_launch/description/bimanual_dexee_ur.urdf.xacro (robot description, xacro)
@@ -50,5 +50,8 @@
   <xacro:include filename="$(find ur_description)/urdf/inc/$(arg arm_model_1)_macro.xacro"/>
   <!-- Include hand description -->
-  <xacro:include filename="$(find dx_description)/robot/$(arg hand_type).xacro" />
+  <xacro:if value="${'$(arg hand_type)' == 'chiral'}">
+    <xacro:include filename="$(find dx_description)/robot/0x02000107.xacro" />
+    <xacro:include filename="$(find dx_description)/robot/0x02000109.xacro" />
+  </xacro:if>
   <!-- ==================== ROBOT SYSTEM 0 ==================== -->
   <xacro:if value="${'$(arg arm_model_0)' == 'ur10e'}">
@@ -64,5 +67,10 @@
       <xacro:ur5_robot prefix="a0_" transmission_hw_interface="$(arg transmission_hw_interface)" kinematics_parameters_file="$(arg kinematics_config_0)"/>
   </xacro:if>
-  <xacro:e3_r3_hand prefix="h0_" />
+  <xacro:if value="${'$(arg hand_type)' == '0x02000105'}">
+      <xacro:dexee_config_1_hand prefix="h0_" />
+  </xacro:if>
+  <xacro:if value="${'$(arg hand_type)' == 'chiral'}">
+      <xacro:dexee_config_2_right_hand prefix="h0_" />
+  </xacro:if>
   <joint name="world_joint_0" type="fixed">
       <parent link="world"/>
@@ -96,5 +104,10 @@
       <xacro:ur5_robot prefix="a1_" transmission_hw_interface="$(arg transmission_hw_interface)" kinematics_parameters_file="$(arg kinematics_config_1)"/>
   </xacro:if>
-  <xacro:e3_r3_hand prefix="h1_" />
+  <xacro:if value="${'$(arg hand_type)' == '0x02000105'}">
+      <xacro:dexee_config_1_hand prefix="h1_" />
+  </xacro:if>
+  <xacro:if value="${'$(arg hand_type)' == 'chiral'}">
+      <xacro:dexee_config_2_left_hand prefix="h1_" />
+  </xacro:if>
   <joint name="world_joint_1" type="fixed">
       <parent link="world"/>
