Commit message: namespaced everything

File: dx_dexee_config_2_lh_moveit_config/config/gazebo_dexee_config_2_left_hand.urdf (robot description, URDF)
Before this commit: robot dexee_config_2_left_hand, 21 links, 20 joints
Links:
- removed link F0_J0_link
- removed link F0_base
- removed link F0_distal
- removed link F0_middle
- removed link F0_proximal
- removed link F0_tip
- removed link F1_J0_link
- removed link F1_base
- removed link F1_distal
- removed link F1_middle
- removed link F1_proximal
- removed link F1_tip
- removed link F2_J0_link
- removed link F2_base
- removed link F2_distal
- removed link F2_middle
- removed link F2_proximal
- removed link F2_tip
- removed link end_effector
- removed link hand_base
- added link h0_F0_J0_link, mass 0.13077995; collision mesh filename=package://dx_description/meshes/dx_e3r3_finger/collision/F0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; visual mesh filename=package://dx_description/meshes/dx_e3r3_finger/F0_J0_link.S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
- added link h0_F0_base, mass 0.89937782; collision mesh filename=package://dx_description/meshes/dx_e3r3_finger/collision/F0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; visual mesh filename=package://dx_description/meshes/dx_e3r3_finger/F0_base.STL
- added link h0_F0_distal, mass 0.02766365; collision mesh filename=package://dx_description/meshes/dx_e3r3_finger/collision/F0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; visual mesh filename=package://dx_description/meshes/dx_e3r3_finger/F0_distal.STL
- added link h0_F0_middle, mass 0.05585897; collision mesh filename=package://dx_description/meshes/dx_e3r3_finger/collision/F0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; visual mesh filename=package://dx_description/meshes/dx_e3r3_finger/F0_middle.STL
- added link h0_F0_proximal, mass 0.09614332; collision mesh filename=package://dx_description/meshes/dx_e3r3_finger/collision/F0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; visual mesh filename=package://dx_description/meshes/dx_e3r3_finger/F0_proximal.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
- added link h0_F0_tip
- added link h0_F1_J0_link, mass 0.13077995; collision mesh filename=package://dx_description/meshes/dx_e3r3_finger/collision/F0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; visual mesh filename=package://dx_description/meshes/dx_e3r3_finger/F0_J0_link.S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
- added link h0_F1_base, mass 0.89937782; collision mesh filename=package://dx_description/meshes/dx_e3r3_finger/collision/F0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; visual mesh filename=package://dx_description/meshes/dx_e3r3_finger/F0_base.STL
- added link h0_F1_distal, mass 0.02766365; collision mesh filename=package://dx_description/meshes/dx_e3r3_finger/collision/F0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; visual mesh filename=package://dx_description/meshes/dx_e3r3_finger/F0_distal.STL
- added link h0_F1_middle, mass 0.05585897; collision mesh filename=package://dx_description/meshes/dx_e3r3_finger/collision/F0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; visual mesh filename=package://dx_description/meshes/dx_e3r3_finger/F0_middle.STL
- added link h0_F1_proximal, mass 0.09614332; collision mesh filename=package://dx_description/meshes/dx_e3r3_finger/collision/F0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; visual mesh filename=package://dx_description/meshes/dx_e3r3_finger/F0_proximal.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
- added link h0_F1_tip
- added link h0_F2_J0_link, mass 0.13077995; collision mesh filename=package://dx_description/meshes/dx_e3r3_finger/collision/F0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; visual mesh filename=package://dx_description/meshes/dx_e3r3_finger/F0_J0_link.S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
- added link h0_F2_base, mass 0.89937782; collision mesh filename=package://dx_description/meshes/dx_e3r3_finger/collision/F0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; visual mesh filename=package://dx_description/meshes/dx_e3r3_finger/F0_base.STL
- added link h0_F2_distal, mass 0.02766365; collision mesh filename=package://dx_description/meshes/dx_e3r3_finger/collision/F0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; visual mesh filename=package://dx_description/meshes/dx_e3r3_finger/F0_distal.STL
- added link h0_F2_middle, mass 0.05585897; collision mesh filename=package://dx_description/meshes/dx_e3r3_finger/collision/F0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; visual mesh filename=package://dx_description/meshes/dx_e3r3_finger/F0_middle.STL
- added link h0_F2_proximal, mass 0.09614332; collision mesh filename=package://dx_description/meshes/dx_e3r3_finger/collision/F0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; visual mesh filename=package://dx_description/meshes/dx_e3r3_finger/F0_proximal.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
- added link h0_F2_tip
- added link h0_end_effector
- added link h0_hand_base, mass 0.53506724; collision mesh filename=package://dx_description/meshes/hand_bases/collision/Config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; visual mesh filename=package://dx_description/meshes/hand_bases/Config_2_Left_Ha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
Joints:
- removed joint F0_J0
- removed joint F0_J1
- removed joint F0_J2
- removed joint F0_J3
- removed joint F0_distal_tip
- removed joint F1_J0
- removed joint F1_J1
- removed joint F1_J2
- removed joint F1_J3
- removed joint F1_distal_tip
- removed joint F2_J0
- removed joint F2_J1
- removed joint F2_J2
- removed joint F2_J3
- removed joint F2_distal_tip
- removed joint ee_fixed_joint
- removed joint world_joint
- removed joint world_joint_F0
- removed joint world_joint_F1
- removed joint world_joint_F2
- added joint h0_F0_J0: type revolute, parent h0_F0_base, child h0_F0_J0_link, origin xyz=0 -0.14073 -0.051327 rpy=2.0944 0 0, axis 0 -1 0, limit lower=-0.8727 upper=0.8727 effort=1.5 velocity=3.1415
- added joint h0_F0_J1: type revolute, parent h0_F0_J0_link, child h0_F0_proximal, origin xyz=0 0.0765883365730207 0.0299999999999999 rpy=0 0 0, axis 1 0 0, limit lower=-1.396 upper=0.785 effort=1.2 velocity=3.1415
- added joint h0_F0_J2: type revolute, parent h0_F0_proximal, child h0_F0_middle, origin xyz=0 0 0.05 rpy=0 0 0, axis 1 0 0, limit lower=0 upper=1.396 effort=0.7 velocity=3.1415
- added joint h0_F0_J3: type revolute, parent h0_F0_middle, child h0_F0_distal, origin xyz=0 0 0.035 rpy=0 0 0, axis 1 0 0, limit lower=-0.523 upper=1.485 effort=0.35 velocity=3.1415
- added joint h0_F0_distal_tip: type fixed, parent h0_F0_distal, child h0_F0_tip, origin xyz=0 0.003 0.033 rpy=0 0 0
- added joint h0_F1_J0: type revolute, parent h0_F1_base, child h0_F1_J0_link, origin xyz=0 -0.14073 -0.051327 rpy=2.0944 0 0, axis 0 -1 0, limit lower=-0.8727 upper=0.8727 effort=1.5 velocity=3.1415
- added joint h0_F1_J1: type revolute, parent h0_F1_J0_link, child h0_F1_proximal, origin xyz=0 0.0765883365730207 0.0299999999999999 rpy=0 0 0, axis 1 0 0, limit lower=-1.396 upper=0.785 effort=1.2 velocity=3.1415
- added joint h0_F1_J2: type revolute, parent h0_F1_proximal, child h0_F1_middle, origin xyz=0 0 0.05 rpy=0 0 0, axis 1 0 0, limit lower=0 upper=1.396 effort=0.7 velocity=3.1415
- added joint h0_F1_J3: type revolute, parent h0_F1_middle, child h0_F1_distal, origin xyz=0 0 0.035 rpy=0 0 0, axis 1 0 0, limit lower=-0.523 upper=1.485 effort=0.35 velocity=3.1415
- added joint h0_F1_distal_tip: type fixed, parent h0_F1_distal, child h0_F1_tip, origin xyz=0 0.003 0.033 rpy=0 0 0
- added joint h0_F2_J0: type revolute, parent h0_F2_base, child h0_F2_J0_link, origin xyz=0 -0.14073 -0.051327 rpy=2.0944 0 0, axis 0 -1 0, limit lower=-0.8727 upper=0.8727 effort=1.5 velocity=3.1415
- added joint h0_F2_J1: type revolute, parent h0_F2_J0_link, child h0_F2_proximal, origin xyz=0 0.0765883365730207 0.0299999999999999 rpy=0 0 0, axis 1 0 0, limit lower=-1.396 upper=0.785 effort=1.2 velocity=3.1415
- added joint h0_F2_J2: type revolute, parent h0_F2_proximal, child h0_F2_middle, origin xyz=0 0 0.05 rpy=0 0 0, axis 1 0 0, limit lower=0 upper=1.396 effort=0.7 velocity=3.1415
- added joint h0_F2_J3: type revolute, parent h0_F2_middle, child h0_F2_distal, origin xyz=0 0 0.035 rpy=0 0 0, axis 1 0 0, limit lower=-0.523 upper=1.485 effort=0.35 velocity=3.1415
- added joint h0_F2_distal_tip: type fixed, parent h0_F2_distal, child h0_F2_tip, origin xyz=0 0.003 0.033 rpy=0 0 0
- added joint h0_ee_fixed_joint: type fixed, parent h0_hand_base, child h0_end_effector, origin xyz=0.0 0.0 0.25 rpy=0.0 0.0 0.0
- added joint h0_world_joint: type fixed, parent world, child h0_hand_base
- added joint h0_world_joint_F0: type fixed, parent h0_hand_base, child h0_F0_base, origin xyz=0 0.05 0.017 rpy=-1.5707 0 0
- added joint h0_world_joint_F1: type fixed, parent h0_hand_base, child h0_F1_base, origin xyz=0.0384 -0.0287 0.017 rpy=-1.5707 0 -2.8159
- added joint h0_world_joint_F2: type fixed, parent h0_hand_base, child h0_F2_base, origin xyz=-0.0384 -0.02870 0.017 rpy=-1.5707 0 2.8159

File: dx_dexee_config_2_rh_moveit_config/config/gazebo_dexee_config_2_right_hand.urdf (robot description, URDF)
Before this commit: robot dexee_config_2_right_hand, 21 links, 20 joints
Links:
- removed link F0_J0_link
- removed link F0_base
- removed link F0_distal
- removed link F0_middle
- removed link F0_proximal
- removed link F0_tip
- removed link F1_J0_link
- removed link F1_base
- removed link F1_distal
- removed link F1_middle
- removed link F1_proximal
- removed link F1_tip
- removed link F2_J0_link
- removed link F2_base
- removed link F2_distal
- removed link F2_middle
- removed link F2_proximal
- removed link F2_tip
- removed link end_effector
- removed link hand_base
- added link h0_F0_J0_link, mass 0.13077995; collision mesh filename=package://dx_description/meshes/dx_e3r3_finger/collision/F0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; visual mesh filename=package://dx_description/meshes/dx_e3r3_finger/F0_J0_link.S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
- added link h0_F0_base, mass 0.89937782; collision mesh filename=package://dx_description/meshes/dx_e3r3_finger/collision/F0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; visual mesh filename=package://dx_description/meshes/dx_e3r3_finger/F0_base.STL
- added link h0_F0_distal, mass 0.02766365; collision mesh filename=package://dx_description/meshes/dx_e3r3_finger/collision/F0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; visual mesh filename=package://dx_description/meshes/dx_e3r3_finger/F0_distal.STL
- added link h0_F0_middle, mass 0.05585897; collision mesh filename=package://dx_description/meshes/dx_e3r3_finger/collision/F0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; visual mesh filename=package://dx_description/meshes/dx_e3r3_finger/F0_middle.STL
- added link h0_F0_proximal, mass 0.09614332; collision mesh filename=package://dx_description/meshes/dx_e3r3_finger/collision/F0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; visual mesh filename=package://dx_description/meshes/dx_e3r3_finger/F0_proximal.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
- added link h0_F0_tip
- added link h0_F1_J0_link, mass 0.13077995; collision mesh filename=package://dx_description/meshes/dx_e3r3_finger/collision/F0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; visual mesh filename=package://dx_description/meshes/dx_e3r3_finger/F0_J0_link.S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
- added link h0_F1_base, mass 0.89937782; collision mesh filename=package://dx_description/meshes/dx_e3r3_finger/collision/F0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; visual mesh filename=package://dx_description/meshes/dx_e3r3_finger/F0_base.STL
- added link h0_F1_distal, mass 0.02766365; collision mesh filename=package://dx_description/meshes/dx_e3r3_finger/collision/F0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; visual mesh filename=package://dx_description/meshes/dx_e3r3_finger/F0_distal.STL
- added link h0_F1_middle, mass 0.05585897; collision mesh filename=package://dx_description/meshes/dx_e3r3_finger/collision/F0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; visual mesh filename=package://dx_description/meshes/dx_e3r3_finger/F0_middle.STL
- added link h0_F1_proximal, mass 0.09614332; collision mesh filename=package://dx_description/meshes/dx_e3r3_finger/collision/F0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; visual mesh filename=package://dx_description/meshes/dx_e3r3_finger/F0_proximal.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
- added link h0_F1_tip
- added link h0_F2_J0_link, mass 0.13077995; collision mesh filename=package://dx_description/meshes/dx_e3r3_finger/collision/F0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; visual mesh filename=package://dx_description/meshes/dx_e3r3_finger/F0_J0_link.S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
- added link h0_F2_base, mass 0.89937782; collision mesh filename=package://dx_description/meshes/dx_e3r3_finger/collision/F0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; visual mesh filename=package://dx_description/meshes/dx_e3r3_finger/F0_base.STL
- added link h0_F2_distal, mass 0.02766365; collision mesh filename=package://dx_description/meshes/dx_e3r3_finger/collision/F0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; visual mesh filename=package://dx_description/meshes/dx_e3r3_finger/F0_distal.STL
- added link h0_F2_middle, mass 0.05585897; collision mesh filename=package://dx_description/meshes/dx_e3r3_finger/collision/F0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; visual mesh filename=package://dx_description/meshes/dx_e3r3_finger/F0_middle.STL
- added link h0_F2_proximal, mass 0.09614332; collision mesh filename=package://dx_description/meshes/dx_e3r3_finger/collision/F0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; visual mesh filename=package://dx_description/meshes/dx_e3r3_finger/F0_proximal.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
- added link h0_F2_tip
- added link h0_end_effector
- added link h0_hand_base, mass 0.53506724; collision mesh filename=package://dx_description/meshes/hand_bases/collision/Config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; visual mesh filename=package://dx_description/meshes/hand_bases/Config_2_Right_H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
Joints:
- removed joint F0_J0
- removed joint F0_J1
- removed joint F0_J2
- removed joint F0_J3
- removed joint F0_distal_tip
- removed joint F1_J0
- removed joint F1_J1
- removed joint F1_J2
- removed joint F1_J3
- removed joint F1_distal_tip
- removed joint F2_J0
- removed joint F2_J1
- removed joint F2_J2
- removed joint F2_J3
- removed joint F2_distal_tip
- removed joint ee_fixed_joint
- removed joint world_joint
- removed joint world_joint_F0
- removed joint world_joint_F1
- removed joint world_joint_F2
- added joint h0_F0_J0: type revolute, parent h0_F0_base, child h0_F0_J0_link, origin xyz=0 -0.14073 -0.051327 rpy=2.0944 0 0, axis 0 -1 0, limit lower=-0.8727 upper=0.8727 effort=1.5 velocity=3.1415
- added joint h0_F0_J1: type revolute, parent h0_F0_J0_link, child h0_F0_proximal, origin xyz=0 0.0765883365730207 0.0299999999999999 rpy=0 0 0, axis 1 0 0, limit lower=-1.396 upper=0.785 effort=1.2 velocity=3.1415
- added joint h0_F0_J2: type revolute, parent h0_F0_proximal, child h0_F0_middle, origin xyz=0 0 0.05 rpy=0 0 0, axis 1 0 0, limit lower=0 upper=1.396 effort=0.7 velocity=3.1415
- added joint h0_F0_J3: type revolute, parent h0_F0_middle, child h0_F0_distal, origin xyz=0 0 0.035 rpy=0 0 0, axis 1 0 0, limit lower=-0.523 upper=1.485 effort=0.35 velocity=3.1415
- added joint h0_F0_distal_tip: type fixed, parent h0_F0_distal, child h0_F0_tip, origin xyz=0 0.003 0.033 rpy=0 0 0
- added joint h0_F1_J0: type revolute, parent h0_F1_base, child h0_F1_J0_link, origin xyz=0 -0.14073 -0.051327 rpy=2.0944 0 0, axis 0 -1 0, limit lower=-0.8727 upper=0.8727 effort=1.5 velocity=3.1415
- added joint h0_F1_J1: type revolute, parent h0_F1_J0_link, child h0_F1_proximal, origin xyz=0 0.0765883365730207 0.0299999999999999 rpy=0 0 0, axis 1 0 0, limit lower=-1.396 upper=0.785 effort=1.2 velocity=3.1415
- added joint h0_F1_J2: type revolute, parent h0_F1_proximal, child h0_F1_middle, origin xyz=0 0 0.05 rpy=0 0 0, axis 1 0 0, limit lower=0 upper=1.396 effort=0.7 velocity=3.1415
- added joint h0_F1_J3: type revolute, parent h0_F1_middle, child h0_F1_distal, origin xyz=0 0 0.035 rpy=0 0 0, axis 1 0 0, limit lower=-0.523 upper=1.485 effort=0.35 velocity=3.1415
- added joint h0_F1_distal_tip: type fixed, parent h0_F1_distal, child h0_F1_tip, origin xyz=0 0.003 0.033 rpy=0 0 0
- added joint h0_F2_J0: type revolute, parent h0_F2_base, child h0_F2_J0_link, origin xyz=0 -0.14073 -0.051327 rpy=2.0944 0 0, axis 0 -1 0, limit lower=-0.8727 upper=0.8727 effort=1.5 velocity=3.1415
- added joint h0_F2_J1: type revolute, parent h0_F2_J0_link, child h0_F2_proximal, origin xyz=0 0.0765883365730207 0.0299999999999999 rpy=0 0 0, axis 1 0 0, limit lower=-1.396 upper=0.785 effort=1.2 velocity=3.1415
- added joint h0_F2_J2: type revolute, parent h0_F2_proximal, child h0_F2_middle, origin xyz=0 0 0.05 rpy=0 0 0, axis 1 0 0, limit lower=0 upper=1.396 effort=0.7 velocity=3.1415
- added joint h0_F2_J3: type revolute, parent h0_F2_middle, child h0_F2_distal, origin xyz=0 0 0.035 rpy=0 0 0, axis 1 0 0, limit lower=-0.523 upper=1.485 effort=0.35 velocity=3.1415
- added joint h0_F2_distal_tip: type fixed, parent h0_F2_distal, child h0_F2_tip, origin xyz=0 0.003 0.033 rpy=0 0 0
- added joint h0_ee_fixed_joint: type fixed, parent h0_hand_base, child h0_end_effector, origin xyz=0.0 0.0 0.25 rpy=0.0 0.0 0.0
- added joint h0_world_joint: type fixed, parent world, child h0_hand_base
- added joint h0_world_joint_F0: type fixed, parent h0_hand_base, child h0_F0_base, origin xyz=0 0.05 0.017 rpy=-1.5707 0 0
- added joint h0_world_joint_F1: type fixed, parent h0_hand_base, child h0_F1_base, origin xyz=0.0384 -0.0287 0.017 rpy=-1.5707 0 -2.8159
- added joint h0_world_joint_F2: type fixed, parent h0_hand_base, child h0_F2_base, origin xyz=-0.0384 -0.02870 0.017 rpy=-1.5707 0 2.8159
